File: hardware/main.brd (EAGLE design)
At the start: 100 x 80 mm, 96 parts, among them IC1 IS61WV102416BLL-10T, U1 LCMXO2-7000HC-4TG144I, U3 W25Q32FV

Commit message: 6MHz TSX3225 replaced with 6x3
Parts:
- X1: value (none) -> CRYSTALS-NOGND-WATCH-3X8; device PP_FreqCtrl:TSX-3225 -> IQD-Frequency-Products:WATCH-3X8
- moved X1 0.51 mm to (83.3, 62.0)
Connections:
- net GND: no longer X1.2, X1.4
- net N$18: now also X1.2; no longer X1.3
Routing:
- net N$18: track 7.18 -> 8.34 mm
Changed lines of the file:
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@@
 <setting verticaltext="up"/>
 </settings>
-<grid distance="20" unitdist="mil" unit="mil" style="lines" multiple="1" display="no" altdistance="5" altunitdist="mil" altunit="mil"/>
+<grid distance="10" unitdist="mil" unit="mil" style="lines" multiple="1" display="no" altdistance="5" altunitdist="mil" altunit="mil"/>
 <layers>
 <layer number="1" name="Top" color="4" fill="1" visible="yes" active="yes"/>
@@
 <vertex x="83.312" y="65.532"/>
 <vertex x="83.566" y="65.278"/>
-<vertex x="83.566" y="62.23"/>
-<vertex x="85.344" y="62.23"/>
+<vertex x="83.566" y="63.754"/>
+<vertex x="85.344" y="63.754"/>
 <vertex x="85.344" y="56.896"/>
 <vertex x="83.566" y="56.896"/>
 <vertex x="83.566" y="58.166"/>
 <vertex x="83.058" y="58.674"/>
-<vertex x="83.058" y="60.706"/>
-<vertex x="81.788" y="60.706"/>
+<vertex x="83.058" y="60.198"/>
+<vertex x="81.788" y="60.198"/>
 <vertex x="81.788" y="59.944"/>
 <vertex x="78.994" y="59.944"/>
@@
 <vertex x="76.708" y="27.432"/>
 <vertex x="76.708" y="30.48"/>
+</polygon>
+<polygon width="0.1524" layer="42">
+<vertex x="78.994" y="59.944"/>
+<vertex x="78.994" y="61.976"/>
+<vertex x="79.502" y="61.976"/>
+<vertex x="79.502" y="62.992"/>
+<vertex x="81.534" y="65.024"/>
+<vertex x="81.534" y="66.04"/>
+<vertex x="83.312" y="66.04"/>
+<vertex x="83.312" y="65.532"/>
+<vertex x="83.566" y="65.278"/>
+<vertex x="83.566" y="63.754"/>
+<vertex x="85.344" y="63.754"/>
+<vertex x="85.344" y="56.896"/>
+<vertex x="83.566" y="56.896"/>
+<vertex x="83.566" y="58.166"/>
+<vertex x="83.058" y="58.674"/>
+<vertex x="83.058" y="60.198"/>
+<vertex x="81.788" y="60.198"/>
+<vertex x="81.788" y="59.944"/>
 </polygon>
 </plain>
@@
 <element name="R10" library="resistor" library_urn="urn:adsk.eagle:library:348" package="R0603" package3d_urn="urn:adsk.eagle:package:26057/1" value="1K" x="36.83" y="22.86" rot="R90"/>
 <element name="U$12" library="mouse_enc" package="SWITCH_6X6" value="SWITCH_6X6" x="41.402" y="5.334"/>
-<element name="X1" library="PP_FreqCtrl" package="TSX-3225" value="" x="83.312" y="61.468" rot="R90"/>
 <element name="Q1" library="crystal-geyer_V1_0" library_urn="urn:adsk.eagle:library:203" package="7.0X5.0_KXO-82-TCXO" package3d_urn="urn:adsk.eagle:package:11956/1" value="" x="32.004" y="46.99"/>
 <element name="R11" library="resistor" library_urn="urn:adsk.eagle:library:348" package="R0603" package3d_urn="urn:adsk.eagle:package:26057/1" value="10" x="38.354" y="48.514" rot="R180"/>
@@
 <element name="C29" library="resistor" library_urn="urn:adsk.eagle:library:348" package="C0603" package3d_urn="urn:adsk.eagle:package:26138/1" value="100nF" x="57.785" y="38.1" rot="MR0"/>
 <element name="JP4" library="pinhead" library_urn="urn:adsk.eagle:library:325" package="1X04" package3d_urn="urn:adsk.eagle:package:22407/2" value="" x="54.61" y="75.565"/>
+<element name="X1" library="IQD-Frequency-Products" library_urn="urn:adsk.eagle:library:90" package="WATCH-3X8" package3d_urn="urn:adsk.eagle:package:3354/1" value="CRYSTALS-NOGND-WATCH-3X8" x="83.312" y="61.976" rot="R90"/>
 </elements>
 <signals>
@@
 <wire x1="73.63" y1="74.77" x2="73.63" y2="75.916" width="0.4064" layer="1"/>
 <wire x1="73.63" y1="75.916" x2="74.169625" y2="76.455625" width="0.4064" layer="1"/>
-<contactref element="X1" pad="2"/>
-<contactref element="X1" pad="4"/>
 <wire x1="72.664" y1="65.21" x2="72.664" y2="66.274" width="0.254" layer="1"/>
 <wire x1="72.664" y1="66.274" x2="72.644" y2="66.294" width="0.254" layer="1"/>
@@
 <wire x1="78.164" y1="61.21" x2="79.672" y2="61.21" width="0.1524" layer="1"/>
 <wire x1="79.672" y1="61.21" x2="80.264" y2="60.618" width="0.1524" layer="1"/>
+<wire x1="80.938" y1="60.618" x2="80.264" y2="60.618" width="0.1524" layer="1"/>
+<wire x1="84.112" y1="57.962" x2="84.162" y2="57.912" width="0.1524" layer="1"/>
 <contactref element="X1" pad="1"/>
-<wire x1="80.264" y1="60.618" x2="80.938" y2="60.618" width="0.1524" layer="1"/>
-<wire x1="80.938" y1="60.618" x2="81.788" y2="61.468" width="0.1524" layer="1"/>
-<wire x1="81.788" y1="61.468" x2="83.012" y2="61.468" width="0.1524" layer="1"/>
-<wire x1="83.012" y1="61.468" x2="84.112" y2="60.368" width="0.1524" layer="1"/>
-<wire x1="84.112" y1="60.368" x2="84.112" y2="57.962" width="0.1524" layer="1"/>
-<wire x1="84.112" y1="57.962" x2="84.162" y2="57.912" width="0.1524" layer="1"/>
+<wire x1="83.312" y1="61.426" x2="81.746" y2="61.426" width="0.1524" layer="1"/>
+<wire x1="81.746" y1="61.426" x2="80.938" y2="60.618" width="0.1524" layer="1"/>
+<wire x1="84.162" y1="57.912" x2="84.162" y2="60.576" width="0.1524" layer="1"/>
+<wire x1="84.162" y1="60.576" x2="83.312" y2="61.426" width="0.1524" layer="1"/>
 </signal>
 <signal name="N$18">
@@
 <wire x1="78.164" y1="61.71" x2="79.656" y2="61.71" width="0.1524" layer="1"/>
 <wire x1="79.656" y1="61.71" x2="80.264" y2="62.318" width="0.1524" layer="1"/>
-<contactref element="X1" pad="3"/>
-<wire x1="80.264" y1="62.318" x2="82.262" y2="62.318" width="0.1524" layer="1"/>
-<wire x1="82.262" y1="62.318" x2="82.512" y2="62.568" width="0.1524" layer="1"/>
-<wire x1="82.512" y1="62.568" x2="82.512" y2="64.974" width="0.1524" layer="1"/>
 <wire x1="82.512" y1="64.974" x2="82.462" y2="65.024" width="0.1524" layer="1"/>
+<contactref element="X1" pad="2"/>
+<wire x1="83.312" y1="62.526" x2="80.472" y2="62.526" width="0.1524" layer="1"/>
+<wire x1="80.472" y1="62.526" x2="80.264" y2="62.318" width="0.1524" layer="1"/>
+<wire x1="83.312" y1="62.526" x2="82.512" y2="63.326" width="0.1524" layer="1"/>
+<wire x1="82.512" y1="63.326" x2="82.512" y2="64.974" width="0.1524" layer="1"/>
 </signal>
 <signal name="+5V">

Commit message: schematic fixes
Parts:
- C17, C18: value 18pF -> 27pF
- R12: value 1M -> DNP
- R47: value 470 -> 1K
Changed lines of the file:
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@@
 <element name="C14" library="resistor" library_urn="urn:adsk.eagle:library:348" package="C0603" package3d_urn="urn:adsk.eagle:package:26138/1" value="100nF" x="81.026" y="68.072" rot="R90"/>
 <element name="C15" library="resistor" library_urn="urn:adsk.eagle:library:348" package="C0603" package3d_urn="urn:adsk.eagle:package:26138/1" value="100nF" x="75.184" y="53.594"/>
-<element name="R12" library="resistor" library_urn="urn:adsk.eagle:library:348" package="R0603" package3d_urn="urn:adsk.eagle:package:26057/1" value="1M" x="80.264" y="61.468" rot="R90"/>
-<element name="C17" library="resistor" library_urn="urn:adsk.eagle:library:348" package="C0603" package3d_urn="urn:adsk.eagle:package:26138/1" value="18pF" x="83.312" y="57.912" rot="R180"/>
-<element name="C18" library="resistor" library_urn="urn:adsk.eagle:library:348" package="C0603" package3d_urn="urn:adsk.eagle:package:26138/1" value="18pF" x="83.312" y="65.024"/>
+<element name="R12" library="resistor" library_urn="urn:adsk.eagle:library:348" package="R0603" package3d_urn="urn:adsk.eagle:package:26057/1" value="DNP" x="80.264" y="61.468" rot="R90"/>
+<element name="C17" library="resistor" library_urn="urn:adsk.eagle:library:348" package="C0603" package3d_urn="urn:adsk.eagle:package:26138/1" value="27pF" x="83.312" y="57.912" rot="R180"/>
+<element name="C18" library="resistor" library_urn="urn:adsk.eagle:library:348" package="C0603" package3d_urn="urn:adsk.eagle:package:26138/1" value="27pF" x="83.312" y="65.024"/>
 <element name="U3" library="SparkFun-IC-Memory" package="SOIC-8" value="W25Q32FV" x="33.274" y="36.449" rot="R180">
 <attribute name="PROD_ID" value="IC-13229" x="33.274" y="36.449" size="1.778" layer="27" rot="R180" display="off"/>
@@
 <element name="R46" library="resistor" library_urn="urn:adsk.eagle:library:348" package="R0603" package3d_urn="urn:adsk.eagle:package:26057/1" value="10K" x="78.105" y="67.945"/>
 <element name="LED2" library="led" library_urn="urn:adsk.eagle:library:259" package="CHIPLED_0603" package3d_urn="urn:adsk.eagle:package:15822/2" value="" x="50.038" y="5.588" rot="R90"/>
-<element name="R47" library="resistor" library_urn="urn:adsk.eagle:library:348" package="R0603" package3d_urn="urn:adsk.eagle:package:26057/1" value="470" x="53.975" y="5.715" rot="R180"/>
+<element name="R47" library="resistor" library_urn="urn:adsk.eagle:library:348" package="R0603" package3d_urn="urn:adsk.eagle:package:26057/1" value="1K" x="53.975" y="5.715" rot="R180"/>
 <element name="C26" library="resistor" library_urn="urn:adsk.eagle:library:348" package="C0603" package3d_urn="urn:adsk.eagle:package:26138/1" value="100nF" x="53.34" y="45.72" rot="MR270"/>
 <element name="C27" library="resistor" library_urn="urn:adsk.eagle:library:348" package="C0603" package3d_urn="urn:adsk.eagle:package:26138/1" value="100nF" x="49.53" y="42.545" rot="MR180"/>

Commit message: 6-bit video dac
Parts:
- R32: value 230 -> DNP
- R33: value 115 -> 0R
Changed lines of the file:
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@@
 <element name="C24" library="SparkFun" package="EIA7343" value="100uF" x="13.335" y="45.085" rot="MR270"/>
 <element name="C25" library="SparkFun" package="EIA7343" value="100uF" x="19.685" y="51.435" rot="MR270"/>
-<element name="R32" library="resistor" library_urn="urn:adsk.eagle:library:348" package="R0603" package3d_urn="urn:adsk.eagle:package:26057/1" value="230" x="43.18" y="59.69" rot="R90"/>
-<element name="R33" library="resistor" library_urn="urn:adsk.eagle:library:348" package="R0603" package3d_urn="urn:adsk.eagle:package:26057/1" value="115" x="40.64" y="59.69" rot="R270"/>
+<element name="R32" library="resistor" library_urn="urn:adsk.eagle:library:348" package="R0603" package3d_urn="urn:adsk.eagle:package:26057/1" value="DNP" x="43.18" y="59.69" rot="R90"/>
+<element name="R33" library="resistor" library_urn="urn:adsk.eagle:library:348" package="R0603" package3d_urn="urn:adsk.eagle:package:26057/1" value="0R" x="40.64" y="59.69" rot="R270"/>
 <element name="R34" library="resistor" library_urn="urn:adsk.eagle:library:348" package="R0603" package3d_urn="urn:adsk.eagle:package:26057/1" value="230" x="38.1" y="59.69" rot="R90"/>
 <element name="R35" library="resistor" library_urn="urn:adsk.eagle:library:348" package="R0603" package3d_urn="urn:adsk.eagle:package:26057/1" value="230" x="33.02" y="59.69" rot="R90"/>

Commit message: Schematic and pcb fixes. Removed vid6 from video dac, io0 from GPIO port. Missed keyboard lines connected: ps2data to vid6, ps2clk to io0
Parts:
- removed R32: DNP, resistor:R0603
- removed R33: 0R, resistor:R0603
- moved LED1 19.6 mm to (50.8, 5.33), turned to 90 degrees
- moved LED2 10.2 mm to (60.2, 5.33), turned to 270 degrees
- moved AUDIO 2.54 mm to (4.45, 58.4)
- moved R47 2.05 mm to (55.8, 6.73), turned to 0 degrees
- moved VIDEO 1.27 mm to (31.8, 69.2)
Connections:
- removed net IO0: JP3.1, U1.2
- removed net N$21: R32.2, R33.1, VIDEO.1
- removed net VID6: R32.1, U1.138
- net GND: now also JP3.1
- net N$25: now also VIDEO.1; no longer R33.2
- net PS2_CLOCK: now also U1.2
- net PS2_DATA: now also U1.138
Routing:
- net IO0: track 45.0 -> 0.00 mm
- net PS2_DATA: track 2.62 -> 45.6 mm, vias 0 -> 1
- net PS2_CLOCK: track 2.62 -> 44.3 mm, vias 0 -> 1
- net N$2: track 2.35 -> 26.7 mm, vias 0 -> 2
- net N$10: track 5.47 -> 27.6 mm, vias 0 -> 2
- net N$5: track 4.27 -> 24.1 mm, vias 0 -> 2
- net N$21: track 13.8 -> 0.00 mm
- net VID6: track 9.92 -> 0.00 mm
- net +3V3: track 534.6 -> 527.3 mm
- net N$25: track 5.78 -> 10.3 mm
- net N$20: track 5.72 -> 7.89 mm
- net N$24: track 14.0 -> 16.0 mm
- net N$32: track 2.39 -> 3.42 mm
- net GND: vias 447 -> 472
